File: distance_meter_hardware/distance_meter_hardware.kicad_pcb (KiCad board)
At the start: 2 copper layers, 95.5 x 55.5 mm, 6 parts, among them J1 PPPC071LFBN-RC, J2 PPPC071LFBN-RC, J3 PPPC141LFBN-RC, J4 PPPC141LFBN-RC, J5 PPPC071LFBN-RC, J6 PPPC071LFBN-RC

Commit message: Add routing to PCB layout
Connections:
- J4 pad 10: Net-(J4-Pad10) -> GND
- J4 pad 11: Net-(J4-Pad11) -> +5V
Routing:
- net Net-(J3-Pad3): track 0.00 -> 34.0 mm
- net Net-(J3-Pad5): track 0.00 -> 29.0 mm
- net Net-(J3-Pad4): track 0.00 -> 27.8 mm
- net Net-(J1-Pad3): track 0.00 -> 27.1 mm
- net Net-(J3-Pad6): track 0.00 -> 24.8 mm
- net Net-(J3-Pad2): track 0.00 -> 17.3 mm
- added copper zone on F.Cu, net +5V
- added copper zone on B.Cu, net GND
Changed lines of the file:
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@@
     (thickness 1.6)
     (drawings 27)
-    (tracks 4)
+    (tracks 22)
     (zones 0)
     (modules 6)
-    (nets 49)
+    (nets 47)
   )
   (page A4)
@@
   )
   (setup
-    (last_trace_width 0.25)
+    (last_trace_width 0.254)
+    (user_trace_width 0.254)
     (trace_clearance 0.2)
     (zone_clearance 0.508)
@@
   (net 33 "Net-(J4-Pad8)")
   (net 34 "Net-(J4-Pad9)")
-  (net 35 "Net-(J4-Pad10)")
-  (net 36 "Net-(J4-Pad11)")
-  (net 37 "Net-(J4-Pad12)")
-  (net 38 "Net-(J4-Pad13)")
-  (net 39 "Net-(J4-Pad14)")
-  (net 40 "Net-(J6-Pad7)")
-  (net 41 "Net-(J6-Pad6)")
-  (net 42 "Net-(J6-Pad5)")
-  (net 43 "Net-(J6-Pad4)")
-  (net 44 "Net-(J6-Pad3)")
-  (net 45 "Net-(J6-Pad2)")
-  (net 46 "Net-(J6-Pad1)")
-  (net 47 GND)
-  (net 48 +5V)
+  (net 35 "Net-(J4-Pad12)")
+  (net 36 "Net-(J4-Pad13)")
+  (net 37 "Net-(J4-Pad14)")
+  (net 38 "Net-(J6-Pad7)")
+  (net 39 "Net-(J6-Pad6)")
+  (net 40 "Net-(J6-Pad5)")
+  (net 41 "Net-(J6-Pad4)")
+  (net 42 "Net-(J6-Pad3)")
+  (net 43 "Net-(J6-Pad2)")
+  (net 44 "Net-(J6-Pad1)")
+  (net 45 GND)
+  (net 46 +5V)
   (net_class Default "This is the default net class."
     (clearance 0.2)
@@
     (add_net "Net-(J3-Pad9)")
     (add_net "Net-(J4-Pad1)")
-    (add_net "Net-(J4-Pad10)")
-    (add_net "Net-(J4-Pad11)")
     (add_net "Net-(J4-Pad12)")
     (add_net "Net-(J4-Pad13)")
@@
     (fp_line (start -9.398 1.524) (end -9.398 -1.524) (layer B.CrtYd) (width 0.05))
     (pad 7 thru_hole circle (at 7.62 0 180) (size 1.52 1.52) (drill 1.02) (layers *.Cu *.Mask)
-      (net 47 GND))
+      (net 45 GND))
     (pad 6 thru_hole circle (at 5.08 0 180) (size 1.52 1.52) (drill 1.02) (layers *.Cu *.Mask)
-      (net 48 +5V))
+      (net 46 +5V))
     (pad 5 thru_hole circle (at 2.54 0 180) (size 1.52 1.52) (drill 1.02) (layers *.Cu *.Mask)
       (net 1 "Net-(J1-Pad5)"))
@@
       (net 34 "Net-(J4-Pad9)"))
     (pad 10 thru_hole circle (at 6.35 0 270) (size 1.52 1.52) (drill 1.02) (layers *.Cu *.Mask)
-      (net 35 "Net-(J4-Pad10)"))
+      (net 45 GND))
     (pad 11 thru_hole circle (at 8.89 0 270) (size 1.52 1.52) (drill 1.02) (layers *.Cu *.Mask)
-      (net 36 "Net-(J4-Pad11)"))
+      (net 46 +5V))
     (pad 12 thru_hole circle (at 11.43 0 270) (size 1.52 1.52) (drill 1.02) (layers *.Cu *.Mask)
-      (net 37 "Net-(J4-Pad12)"))
+      (net 35 "Net-(J4-Pad12)"))
     (pad 13 thru_hole circle (at 13.97 0 270) (size 1.52 1.52) (drill 1.02) (layers *.Cu *.Mask)
-      (net 38 "Net-(J4-Pad13)"))
+      (net 36 "Net-(J4-Pad13)"))
     (pad 14 thru_hole circle (at 16.51 0 270) (size 1.52 1.52) (drill 1.02) (layers *.Cu *.Mask)
-      (net 39 "Net-(J4-Pad14)"))
+      (net 37 "Net-(J4-Pad14)"))
     (model ${KISYS3DMOD}/Connector_PinSocket_2.54mm.3dshapes/PinSocket_1x14_P2.54mm_Vertical.step
       (offset (xyz 16.76 0 0))
@@
       (net 23 "Net-(J3-Pad4)"))
     (pad 6 thru_hole circle (at 5.08 0 180) (size 1.52 1.52) (drill 1.02) (layers *.Cu *.Mask)
-      (net 48 +5V))
+      (net 46 +5V))
     (pad 7 thru_hole circle (at 7.62 0 180) (size 1.52 1.52) (drill 1.02) (layers *.Cu *.Mask)
-      (net 47 GND))
+      (net 45 GND))
     (model ${KISYS3DMOD}/Connector_PinSocket_2.54mm.3dshapes/PinSocket_1x07_P2.54mm_Vertical.step
       (offset (xyz 7.62 0 0))
@@
     (fp_line (start -9.398 1.524) (end -9.398 -1.524) (layer B.CrtYd) (width 0.05))
     (pad 7 thru_hole circle (at 7.62 0 180) (size 1.52 1.52) (drill 1.02) (layers *.Cu *.Mask)
-      (net 40 "Net-(J6-Pad7)"))
+      (net 38 "Net-(J6-Pad7)"))
     (pad 6 thru_hole circle (at 5.08 0 180) (size 1.52 1.52) (drill 1.02) (layers *.Cu *.Mask)
-      (net 41 "Net-(J6-Pad6)"))
+      (net 39 "Net-(J6-Pad6)"))
     (pad 5 thru_hole circle (at 2.54 0 180) (size 1.52 1.52) (drill 1.02) (layers *.Cu *.Mask)
-      (net 42 "Net-(J6-Pad5)"))
+      (net 40 "Net-(J6-Pad5)"))
     (pad 4 thru_hole circle (at 0 0 180) (size 1.52 1.52) (drill 1.02) (layers *.Cu *.Mask)
-      (net 43 "Net-(J6-Pad4)"))
+      (net 41 "Net-(J6-Pad4)"))
     (pad 3 thru_hole circle (at -2.54 0 180) (size 1.52 1.52) (drill 1.02) (layers *.Cu *.Mask)
-      (net 44 "Net-(J6-Pad3)"))
+      (net 42 "Net-(J6-Pad3)"))
     (pad 2 thru_hole circle (at -5.08 0 180) (size 1.52 1.52) (drill 1.02) (layers *.Cu *.Mask)
-      (net 45 "Net-(J6-Pad2)"))
+      (net 43 "Net-(J6-Pad2)"))
     (pad 1 thru_hole rect (at -7.62 0 180) (size 1.52 1.52) (drill 1.02) (layers *.Cu *.Mask)
-      (net 46 "Net-(J6-Pad1)"))
+      (net 44 "Net-(J6-Pad1)"))
     (model ${KISYS3DMOD}/Connector_PinSocket_2.54mm.3dshapes/PinSocket_1x07_P2.54mm_Vertical.step
       (offset (xyz 7.62 0 0))
@@
   (via (at 62.17 92.77) (size 5.4) (drill 2.85) (layers F.Cu B.Cu) (net 0))
   (via (at 62.17 44.77) (size 5.4) (drill 2.85) (layers F.Cu B.Cu) (net 0))
+  (segment (start 136.860005 64.96) (end 141.8 60.020005) (width 0.254) (layer F.Cu) (net 3))
+  (segment (start 116.71 64.96) (end 136.860005 64.96) (width 0.254) (layer F.Cu) (net 3))
+  (segment (start 88.93 64.96) (end 101.47 64.96) (width 0.254) (layer B.Cu) (net 21))
+  (segment (start 80.27 56.3) (end 88.93 64.96) (width 0.254) (layer B.Cu) (net 21))
+  (segment (start 92.07 53.02) (end 101.47 62.42) (width 0.254) (layer B.Cu) (net 22))
+  (segment (start 77.73 56.3) (end 81.01 53.02) (width 0.254) (layer B.Cu) (net 22))
+  (segment (start 81.01 53.02) (end 92.07 53.02) (width 0.254) (layer B.Cu) (net 22))
+  (segment (start 78.77 59.88) (end 101.47 59.88) (width 0.254) (layer F.Cu) (net 23))
+  (segment (start 75.19 56.3) (end 78.77 59.88) (width 0.254) (layer F.Cu) (net 23))
+  (segment (start 82.81 56.3) (end 89.59 49.52) (width 0.254) (layer F.Cu) (net 24))
+  (segment (start 89.59 49.52) (end 102.42 49.52) (width 0.254) (layer F.Cu) (net 24))
+  (segment (start 101.47 57.34) (end 103.6 57.34) (width 0.254) (layer F.Cu) (net 24))
+  (segment (start 103.6 57.34) (end 104.92 56.02) (width 0.254) (layer F.Cu) (net 24))
+  (segment (start 104.92 52.02) (end 102.42 49.52) (width 0.254) (layer F.Cu) (net 24))
+  (segment (start 104.92 56.02) (end 104.92 52.02) (width 0.254) (layer F.Cu) (net 24))
+  (segment (start 85.35 55.286) (end 85.35 56.3) (width 0.254) (layer F.Cu) (net 26))
+  (segment (start 85.836 54.8) (end 85.35 55.286) (width 0.254) (layer F.Cu) (net 26))
+  (segment (start 101.47 54.8) (end 85.836 54.8) (width 0.254) (layer F.Cu) (net 26))
+  (zone (net 46) (net_name +5V) (layer F.Cu) (hatch edge 0.508)
+    (connect_pads (clearance 0.508))
+    (min_thickness 0.254)
+    (fill yes (arc_segments 32) (thermal_gap 0.508) (thermal_bridge_width 0.508))
+    (polygon
+      (pts
+        (xy 58.42 41.02) (xy 153.92 41.02) (xy 153.92 96.52) (xy 58.42 96.52)
+      )
+    )
+  )
+  (zone (net 45) (net_name GND) (layer B.Cu) (hatch edge 0.508)
+    (connect_pads (clearance 0.508))
+    (min_thickness 0.254)
+    (fill yes (arc_segments 32) (thermal_gap 0.508) (thermal_bridge_width 0.508))
+    (polygon
+      (pts
+        (xy 58.42 41.02) (xy 153.92 41.02) (xy 153.92 96.52) (xy 58.42 96.52)
+      )
+    )
+  )
 )

Commit message: Correct routing
Connections:
- J5 pad 1: Net-(J3-Pad2) -> Net-(J3-Pad13)
- J5 pad 2: Net-(J3-Pad3) -> Net-(J3-Pad12)
- J5 pad 3: Net-(J3-Pad6) -> Net-(J3-Pad9)
- J5 pad 4: Net-(J3-Pad5) -> Net-(J3-Pad10)
- J5 pad 5: Net-(J3-Pad4) -> Net-(J3-Pad11)
Routing:
- net Net-(J3-Pad13): track 0.00 -> 57.3 mm
- net Net-(J3-Pad11): track 0.00 -> 35.1 mm
- net Net-(J3-Pad3): track 34.0 -> 0.00 mm
- net Net-(J3-Pad12): track 0.00 -> 31.6 mm
- net Net-(J3-Pad10): track 0.00 -> 31.5 mm
- net Net-(J3-Pad5): track 29.0 -> 0.00 mm
- net Net-(J3-Pad9): track 0.00 -> 27.9 mm
- net Net-(J3-Pad4): track 27.8 -> 0.00 mm
- net Net-(J3-Pad6): track 24.8 -> 0.00 mm
- net Net-(J3-Pad2): track 17.3 -> 0.00 mm
Changed lines of the file:
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@@
     (thickness 1.6)
     (drawings 27)
-    (tracks 22)
+    (tracks 20)
     (zones 0)
     (modules 6)
@@
     (fp_poly (pts (xy -9.14 -1.27) (xy 9.14 -1.27) (xy 9.14 1.27) (xy -9.14 1.27)) (layer F.Fab) (width 0.05))
     (pad 1 thru_hole rect (at -7.62 0 180) (size 1.52 1.52) (drill 1.02) (layers *.Cu *.Mask)
-      (net 26 "Net-(J3-Pad2)"))
+      (net 14 "Net-(J3-Pad13)"))
     (pad 2 thru_hole circle (at -5.08 0 180) (size 1.52 1.52) (drill 1.02) (layers *.Cu *.Mask)
-      (net 24 "Net-(J3-Pad3)"))
+      (net 15 "Net-(J3-Pad12)"))
     (pad 3 thru_hole circle (at -2.54 0 180) (size 1.52 1.52) (drill 1.02) (layers *.Cu *.Mask)
-      (net 21 "Net-(J3-Pad6)"))
+      (net 18 "Net-(J3-Pad9)"))
     (pad 4 thru_hole circle (at 0 0 180) (size 1.52 1.52) (drill 1.02) (layers *.Cu *.Mask)
-      (net 22 "Net-(J3-Pad5)"))
+      (net 17 "Net-(J3-Pad10)"))
     (pad 5 thru_hole circle (at 2.54 0 180) (size 1.52 1.52) (drill 1.02) (layers *.Cu *.Mask)
-      (net 23 "Net-(J3-Pad4)"))
+      (net 16 "Net-(J3-Pad11)"))
     (pad 6 thru_hole circle (at 5.08 0 180) (size 1.52 1.52) (drill 1.02) (layers *.Cu *.Mask)
       (net 46 +5V))
@@
     )
   )
+  (gr_poly (pts (xy 100.2 47.18) (xy 117.98 47.18) (xy 117.98 90.36) (xy 100.2 90.36)) (layer F.Fab) (width 0.1))
   (dimension 55.5 (width 0.15) (layer F.SilkS)
     (gr_text "55.500 mm" (at 40.12 68.77 90) (layer F.SilkS)
@@
     (arrow2b (pts (xy 58.42 102.02) (xy 59.546504 101.433579)))
   )
-  (gr_poly (pts (xy 100.2 47.18) (xy 117.98 47.18) (xy 117.98 90.36) (xy 100.2 90.36)) (layer F.Fab) (width 0.1))
   (gr_text "SSD1306 OLED LCD" (at 93.224 69.024 270) (layer F.SilkS)
     (effects (font (size 1 1) (thickness 0.15)))
@@
   (segment (start 136.860005 64.96) (end 141.8 60.020005) (width 0.254) (layer F.Cu) (net 3))
   (segment (start 116.71 64.96) (end 136.860005 64.96) (width 0.254) (layer F.Cu) (net 3))
-  (segment (start 88.93 64.96) (end 101.47 64.96) (width 0.254) (layer B.Cu) (net 21))
-  (segment (start 80.27 56.3) (end 88.93 64.96) (width 0.254) (layer B.Cu) (net 21))
-  (segment (start 92.07 53.02) (end 101.47 62.42) (width 0.254) (layer B.Cu) (net 22))
-  (segment (start 77.73 56.3) (end 81.01 53.02) (width 0.254) (layer B.Cu) (net 22))
-  (segment (start 81.01 53.02) (end 92.07 53.02) (width 0.254) (layer B.Cu) (net 22))
-  (segment (start 78.77 59.88) (end 101.47 59.88) (width 0.254) (layer F.Cu) (net 23))
-  (segment (start 75.19 56.3) (end 78.77 59.88) (width 0.254) (layer F.Cu) (net 23))
-  (segment (start 82.81 56.3) (end 89.59 49.52) (width 0.254) (layer F.Cu) (net 24))
-  (segment (start 89.59 49.52) (end 102.42 49.52) (width 0.254) (layer F.Cu) (net 24))
-  (segment (start 101.47 57.34) (end 103.6 57.34) (width 0.254) (layer F.Cu) (net 24))
-  (segment (start 103.6 57.34) (end 104.92 56.02) (width 0.254) (layer F.Cu) (net 24))
-  (segment (start 104.92 52.02) (end 102.42 49.52) (width 0.254) (layer F.Cu) (net 24))
-  (segment (start 104.92 56.02) (end 104.92 52.02) (width 0.254) (layer F.Cu) (net 24))
-  (segment (start 85.35 55.286) (end 85.35 56.3) (width 0.254) (layer F.Cu) (net 26))
-  (segment (start 85.836 54.8) (end 85.35 55.286) (width 0.254) (layer F.Cu) (net 26))
-  (segment (start 101.47 54.8) (end 85.836 54.8) (width 0.254) (layer F.Cu) (net 26))
+  (segment (start 85.35 55.286) (end 90.616 50.02) (width 0.254) (layer F.Cu) (net 14))
+  (segment (start 85.35 56.3) (end 85.35 55.286) (width 0.254) (layer F.Cu) (net 14))
+  (segment (start 90.616 50.02) (end 103.42 50.02) (width 0.254) (layer F.Cu) (net 14))
+  (segment (start 103.42 50.02) (end 106.42 53.02) (width 0.254) (layer F.Cu) (net 14))
+  (segment (start 106.42 77.79) (end 101.47 82.74) (width 0.254) (layer F.Cu) (net 14))
+  (segment (start 106.42 53.02) (end 106.42 77.79) (width 0.254) (layer F.Cu) (net 14))
+  (segment (start 82.81 61.54) (end 82.81 56.3) (width 0.254) (layer B.Cu) (net 15))
+  (segment (start 101.47 80.2) (end 82.81 61.54) (width 0.254) (layer B.Cu) (net 15))
+  (segment (start 96.55 77.66) (end 75.19 56.3) (width 0.254) (layer F.Cu) (net 16))
+  (segment (start 101.47 77.66) (end 96.55 77.66) (width 0.254) (layer F.Cu) (net 16))
+  (segment (start 96.55 75.12) (end 77.73 56.3) (width 0.254) (layer F.Cu) (net 17))
+  (segment (start 101.47 75.12) (end 96.55 75.12) (width 0.254) (layer F.Cu) (net 17))
+  (segment (start 96.55 72.58) (end 80.27 56.3) (width 0.254) (layer F.Cu) (net 18))
+  (segment (start 101.47 72.58) (end 96.55 72.58) (width 0.254) (layer F.Cu) (net 18))
   (zone (net 46) (net_name +5V) (layer F.Cu) (hatch edge 0.508)
     (connect_pads (clearance 0.508))
